File: hardware/fabfm.brd (EAGLE design)
At the start: 76 x 76 mm, 36 parts, among them J1 POWER_JACKPTH_LOCK, J2 AVR_SPI_PRG_6PTH, U1 LM386, U2 Encoder, U5 V_REG_317SINK

Commit message: v11
-fixed silk mistake
-added locking FP for radio module
Parts:
- JP2: value M10" -> M10LOCK; device SparkFun-Connectors:1X10 -> SparkFun-Connectors:1X10_LOCK
Other:
- board text added: "v11"
- board text removed: "FM Radio Kit"
- board text removed: "v10"
Changed lines of the file:
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@@
 <?xml version="1.0" encoding="utf-8"?>
 <!DOCTYPE eagle SYSTEM "eagle.dtd">
-<eagle version="6.2">
+<eagle version="6.3">
 <drawing>
 <settings>
@@
 <wire x1="67.31" y1="26.67" x2="67.31" y2="41.91" width="0.254" layer="21"/>
 <text x="35.19" y="-5.54" size="1.778" layer="51" font="vector" ratio="15">BACK</text>
-<text x="74.897" y="49.843" size="1.778" layer="16" font="vector" ratio="20" rot="SMR270">v10</text>
+<text x="74.897" y="49.843" size="1.778" layer="16" font="vector" ratio="20" rot="SMR270">v11</text>
 <text x="35.369" y="66.735" size="1.016" layer="21" font="vector" ratio="15">speaker</text>
 <text x="31.115" y="62.23" size="2.1844" layer="21" font="vector" ratio="15">+</text>
@@
 <rectangle x1="19.693115625" y1="51.5856625" x2="19.727403125" y2="51.59709375" layer="21"/>
 <rectangle x1="12.674390625" y1="51.59709375" x2="12.685821875" y2="51.608525" layer="21"/>
-<text x="3.81" y="54.61" size="1.9304" layer="29" font="vector" ratio="20">FM Radio Kit</text>
 <rectangle x1="4.87759375" y1="54.71715625" x2="5.35384375" y2="54.75684375" layer="21"/>
 <rectangle x1="24.08634375" y1="54.71715625" x2="24.56259375" y2="54.75684375" layer="21"/>
@@
 </class>
 </classes>
-<designrules>
+<designrules name="default">
 <description language="en">&lt;b&gt;EAGLE Design Rules&lt;/b&gt;
 &lt;p&gt;
@@
 </element>
 <element name="JP9" library="SparkFun" package="SFE-NEW-WEBLOGO" value="LOGO-SFENEW" x="50.927" y="7.747" smashed="yes"/>
-<element name="JP2" library="SparkFun-Connectors" package="1X10" value="M10&quot;" x="1.27" y="8.89" smashed="yes" rot="R90">
+<element name="JP2" library="SparkFun-Connectors" package="1X10_LOCK" value="M10LOCK" x="1.27" y="8.89" smashed="yes" rot="R90">
 <attribute name="NAME" x="-0.5588" y="7.5438" size="1.27" layer="25" ratio="10" rot="R90"/>
 <attribute name="VALUE" x="4.445" y="7.62" size="1.27" layer="27" rot="R90"/>
@@
 <wire x1="7.62" y1="24.13" x2="7.62" y2="31.623" width="0.4064" layer="1"/>
 <wire x1="7.62" y1="31.623" x2="9.017" y2="33.02" width="0.4064" layer="1"/>
-<wire x1="1.27" y1="24.13" x2="7.62" y2="24.13" width="0.4064" layer="1"/>
+<wire x1="1.143" y1="24.13" x2="7.62" y2="24.13" width="0.4064" layer="1"/>
 <contactref element="IC2" pad="21"/>
 <contactref element="IC2" pad="7"/>
@@
 <wire x1="12.954" y1="38.862" x2="12.319" y2="38.227" width="0.4064" layer="16"/>
 <wire x1="12.319" y1="38.227" x2="12.319" y2="32.639" width="0.4064" layer="16"/>
-<wire x1="12.319" y1="32.639" x2="1.27" y2="21.59" width="0.4064" layer="16"/>
+<wire x1="12.319" y1="32.639" x2="1.397" y2="21.59" width="0.4064" layer="16"/>
 </signal>
 <signal name="SCL">
@@
 <wire x1="13.97" y1="33.02" x2="13.97" y2="37.211" width="0.4064" layer="16"/>
 <wire x1="13.97" y1="33.02" x2="13.97" y2="31.75" width="0.4064" layer="16"/>
-<wire x1="13.97" y1="31.75" x2="1.27" y2="19.05" width="0.4064" layer="16"/>
+<wire x1="13.97" y1="31.75" x2="1.143" y2="19.05" width="0.4064" layer="16"/>
 </signal>
 <signal name="DTR">
@@
 <wire x1="10.16" y1="27.94" x2="10.16" y2="19.05" width="0.4064" layer="1"/>
 <wire x1="10.16" y1="19.05" x2="8.89" y2="17.78" width="0.4064" layer="1"/>
-<wire x1="1.27" y1="13.97" x2="5.08" y2="13.97" width="0.4064" layer="1"/>
+<wire x1="1.143" y1="13.97" x2="5.08" y2="13.97" width="0.4064" layer="1"/>
 <wire x1="5.08" y1="13.97" x2="8.89" y2="17.78" width="0.4064" layer="1"/>
 <wire x1="22.86" y1="31.75" x2="23.6855" y2="31.75" width="0.4064" layer="1"/>
@@
 <contactref element="JP2" pad="9"/>
 <contactref element="JP2" pad="10"/>
-<wire x1="1.27" y1="29.21" x2="1.27" y2="31.75" width="0.4064" layer="1"/>
+<wire x1="1.143" y1="29.21" x2="1.397" y2="31.75" width="0.4064" layer="1"/>
 <wire x1="27.94" y1="45.72" x2="12.7" y2="45.72" width="0.4064" layer="16"/>
 <wire x1="12.7" y1="45.72" x2="1.27" y2="34.29" width="0.4064" layer="16"/>
-<wire x1="1.27" y1="34.29" x2="1.27" y2="31.75" width="0.4064" layer="16"/>
+<wire x1="1.27" y1="34.29" x2="1.397" y2="31.75" width="0.4064" layer="16"/>
 </signal>
 <signal name="A">
@@
 </signal>
 </signals>
-<errors>
-</errors>
 </board>
 </drawing>
